File: reverse-mount-led-keboard.kicad_pcb (KiCad board)
At the start: 2 copper layers, 83.8 x 57.1 mm, 29 parts, among them SW1 SW_PUSH, SW10 SW_PUSH, SW2 SW_PUSH, SW3 SW_PUSH, SW4 SW_PUSH, SW5 SW_PUSH, SW6 SW_PUSH, SW7 SW_PUSH, SW8 SW_PUSH, SW9 SW_PUSH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

Commit message: init
Routing:
- net row1: track 70.0 -> 70.8 mm
- net row2: track 92.7 -> 93.4 mm
- net row0: track 53.5 -> 54.3 mm
