File: reverse-mount-led-keboard.kicad_sch (KiCad schematic)
At the start: 29 parts, among them SW1 SW_PUSH, SW10 SW_PUSH, SW2 SW_PUSH, SW3 SW_PUSH, SW4 SW_PUSH, SW5 SW_PUSH, SW6 SW_PUSH, SW7 SW_PUSH, SW8 SW_PUSH, SW9 SW_PUSH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

Commit message: add firmware
Connections:
- net col0: now also SW1.1, SW4.1, SW7.1, U1.7 (4/D4); no longer D1.1 (K), D2.1 (K), D3.1 (K), U1.8 (5/C6)
- net col1: now also SW2.1, SW5.1, SW8.1, U1.9 (6/D7); no longer D4.1 (K), D5.1 (K), D6.1 (K), U1.10 (7/E6)
- net col2: now also SW3.1, SW6.1, SW9.1, U1.12 (9/B5); no longer D7.1 (K), D8.1 (K), D9.1 (K), U1.11 (8/B4)
- net row0: now also D1.1 (K), D2.1 (K), D3.1 (K), U1.8 (5/C6); no longer SW1.1, SW4.1, SW7.1, U1.7 (4/D4)
- net row1: now also D4.1 (K), D5.1 (K), D6.1 (K), U1.10 (7/E6); no longer SW2.1, SW5.1, SW8.1, U1.9 (6/D7)
- net row2: now also D7.1 (K), D8.1 (K), D9.1 (K), U1.11 (8/B4); no longer SW3.1, SW6.1, SW9.1, U1.12 (9/B5)
Changed lines of the file:
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@@
   (junction (at 147.32 72.39) (diameter 0) (color 0 0 0 0)
   )
+  (junction (at 187.96 54.61) (diameter 0) (color 0 0 0 0)
+  )
   (junction (at 172.72 72.39) (diameter 0) (color 0 0 0 0)
   )
@@
   (junction (at 44.45 114.3) (diameter 0) (color 0 0 0 0)
   )
+  (junction (at 187.96 80.01) (diameter 0) (color 0 0 0 0)
+  )
   (junction (at 198.12 46.99) (diameter 0) (color 0 0 0 0)
   )
@@
   (junction (at 62.23 132.08) (diameter 0) (color 0 0 0 0)
   )
-  (junction (at 187.96 80.01) (diameter 0) (color 0 0 0 0)
-  )
   (junction (at 80.01 165.1) (diameter 0) (color 0 0 0 0)
   )
@@
   )
   (junction (at 62.23 114.3) (diameter 0) (color 0 0 0 0)
-  )
-  (junction (at 187.96 54.61) (diameter 0) (color 0 0 0 0)
   )
   (junction (at 44.45 157.48) (diameter 0) (color 0 0 0 0)
@@
     (stroke (width 0) (type default) (color 0 0 0 0))
   )
-  (wire (pts (xy 187.96 80.01) (xy 187.96 78.74))
-    (stroke (width 0) (type default) (color 0 0 0 0))
-  )
-  (wire (pts (xy 187.96 54.61) (xy 187.96 53.34))
-    (stroke (width 0) (type default) (color 0 0 0 0))
-  )
   (wire (pts (xy 80.01 182.88) (xy 102.87 182.88))
     (stroke (width 0) (type default) (color 0 0 0 0))
@@
     (stroke (width 0) (type default) (color 0 0 0 0))
   )
+  (wire (pts (xy 162.56 80.01) (xy 187.96 80.01))
+    (stroke (width 0) (type default) (color 0 0 0 0))
+  )
+  (wire (pts (xy 147.32 31.75) (xy 147.32 46.99))
+    (stroke (width 0) (type default) (color 0 0 0 0))
+  )
+  (wire (pts (xy 62.23 165.1) (xy 80.01 165.1))
+    (stroke (width 0) (type default) (color 0 0 0 0))
+  )
+  (wire (pts (xy 172.72 46.99) (xy 172.72 72.39))
+    (stroke (width 0) (type default) (color 0 0 0 0))
+  )
+  (wire (pts (xy 162.56 54.61) (xy 187.96 54.61))
+    (stroke (width 0) (type default) (color 0 0 0 0))
+  )
   (wire (pts (xy 187.96 80.01) (xy 213.36 80.01))
     (stroke (width 0) (type default) (color 0 0 0 0))
   )
-  (wire (pts (xy 147.32 31.75) (xy 147.32 46.99))
-    (stroke (width 0) (type default) (color 0 0 0 0))
-  )
-  (wire (pts (xy 62.23 165.1) (xy 80.01 165.1))
-    (stroke (width 0) (type default) (color 0 0 0 0))
-  )
-  (wire (pts (xy 172.72 46.99) (xy 172.72 72.39))
-    (stroke (width 0) (type default) (color 0 0 0 0))
-  )
-  (wire (pts (xy 162.56 54.61) (xy 187.96 54.61))
-    (stroke (width 0) (type default) (color 0 0 0 0))
-  )
   (wire (pts (xy 162.56 109.22) (xy 187.96 109.22))
     (stroke (width 0) (type default) (color 0 0 0 0))
@@
     (stroke (width 0) (type default) (color 0 0 0 0))
   )
-  (wire (pts (xy 162.56 80.01) (xy 187.96 80.01))
-    (stroke (width 0) (type default) (color 0 0 0 0))
-  )
   (wire (pts (xy 31.75 132.08) (xy 44.45 132.08))
     (stroke (width 0) (type default) (color 0 0 0 0))
   )
-  (global_label "col0" (shape input) (at 35.56 50.8 180) (fields_autoplaced)
-    (effects (font (size 1.27 1.27)) (justify right))
-    (property "Intersheet References" "${INTERSHEET_REFS}" (id 0) (at 29.0345 50.8794 0)
-      (effects (font (size 1.27 1.27)) (justify right) hide)
-    )
-  )
-  (global_label "row1" (shape input) (at 172.72 31.75 90) (fields_autoplaced)
+  (global_label "row0" (shape input) (at 35.56 50.8 180) (fields_autoplaced)
+    (effects (font (size 1.27 1.27)) (justify right))
+    (property "Intersheet References" "${INTERSHEET_REFS}" (id 0) (at 28.6717 50.7206 0)
+      (effects (font (size 1.27 1.27)) (justify right) hide)
+    )
+  )
+  (global_label "col1" (shape input) (at 172.72 31.75 90) (fields_autoplaced)
     (effects (font (size 1.27 1.27)) (justify left))
-    (property "Intersheet References" "${INTERSHEET_REFS}" (id 0) (at 172.6406 24.8617 90)
+    (property "Intersheet References" "${INTERSHEET_REFS}" (id 0) (at 172.6406 25.2245 90)
       (effects (font (size 1.27 1.27)) (justify left) hide)
     )
   )
-  (global_label "col0" (shape input) (at 129.54 54.61 180) (fields_autoplaced)
-    (effects (font (size 1.27 1.27)) (justify right))
-    (property "Intersheet References" "${INTERSHEET_REFS}" (id 0) (at 123.0145 54.5306 0)
-      (effects (font (size 1.27 1.27)) (justify right) hide)
-    )
-  )
-  (global_label "row1" (shape input) (at 35.56 53.34 180) (fields_autoplaced)
-    (effects (font (size 1.27 1.27)) (justify right))
-    (property "Intersheet References" "${INTERSHEET_REFS}" (id 0) (at 28.6717 53.4194 0)
-      (effects (font (size 1.27 1.27)) (justify right) hide)
-    )
-  )
-  (global_label "col1" (shape input) (at 129.54 80.01 180) (fields_autoplaced)
-    (effects (font (size 1.27 1.27)) (justify right))
-    (property "Intersheet References" "${INTERSHEET_REFS}" (id 0) (at 123.0145 79.9306 0)
-      (effects (font (size 1.27 1.27)) (justify right) hide)
-    )
-  )
-  (global_label "row2" (shape input) (at 198.12 31.75 90) (fields_autoplaced)
+  (global_label "row0" (shape input) (at 129.54 54.61 180) (fields_autoplaced)
+    (effects (font (size 1.27 1.27)) (justify right))
+    (property "Intersheet References" "${INTERSHEET_REFS}" (id 0) (at 122.6517 54.5306 0)
+      (effects (font (size 1.27 1.27)) (justify right) hide)
+    )
+  )
+  (global_label "col1" (shape input) (at 35.56 53.34 180) (fields_autoplaced)
+    (effects (font (size 1.27 1.27)) (justify right))
+    (property "Intersheet References" "${INTERSHEET_REFS}" (id 0) (at 29.0345 53.2606 0)
+      (effects (font (size 1.27 1.27)) (justify right) hide)
+    )
+  )
+  (global_label "row1" (shape input) (at 129.54 80.01 180) (fields_autoplaced)
+    (effects (font (size 1.27 1.27)) (justify right))
+    (property "Intersheet References" "${INTERSHEET_REFS}" (id 0) (at 122.6517 79.9306 0)
+      (effects (font (size 1.27 1.27)) (justify right) hide)
+    )
+  )
+  (global_label "col2" (shape input) (at 198.12 31.75 90) (fields_autoplaced)
     (effects (font (size 1.27 1.27)) (justify left))
-    (property "Intersheet References" "${INTERSHEET_REFS}" (id 0) (at 198.0406 24.8617 90)
+    (property "Intersheet References" "${INTERSHEET_REFS}" (id 0) (at 198.0406 25.2245 90)
       (effects (font (size 1.27 1.27)) (justify left) hide)
     )
   )
-  (global_label "col2" (shape input) (at 35.56 58.42 180) (fields_autoplaced)
-    (effects (font (size 1.27 1.27)) (justify right))
-    (property "Intersheet References" "${INTERSHEET_REFS}" (id 0) (at 29.0345 58.4994 0)
-      (effects (font (size 1.27 1.27)) (justify right) hide)
-    )
-  )
-  (global_label "row0" (shape input) (at 147.32 31.75 90) (fields_autoplaced)
+  (global_label "row2" (shape input) (at 35.56 58.42 180) (fields_autoplaced)
+    (effects (font (size 1.27 1.27)) (justify right))
+    (property "Intersheet References" "${INTERSHEET_REFS}" (id 0) (at 28.6717 58.3406 0)
+      (effects (font (size 1.27 1.27)) (justify right) hide)
+    )
+  )
+  (global_label "col0" (shape input) (at 147.32 31.75 90) (fields_autoplaced)
     (effects (font (size 1.27 1.27)) (justify left))
-    (property "Intersheet References" "${INTERSHEET_REFS}" (id 0) (at 147.2406 24.8617 90)
+    (property "Intersheet References" "${INTERSHEET_REFS}" (id 0) (at 147.2406 25.2245 90)
       (effects (font (size 1.27 1.27)) (justify left) hide)
     )
   )
-  (global_label "row0" (shape input) (at 35.56 48.26 180) (fields_autoplaced)
-    (effects (font (size 1.27 1.27)) (justify right))
-    (property "Intersheet References" "${INTERSHEET_REFS}" (id 0) (at 28.6717 48.3394 0)
-      (effects (font (size 1.27 1.27)) (justify right) hide)
-    )
-  )
-  (global_label "row2" (shape input) (at 35.56 60.96 180) (fields_autoplaced)
-    (effects (font (size 1.27 1.27)) (justify right))
-    (property "Intersheet References" "${INTERSHEET_REFS}" (id 0) (at 28.6717 60.8806 0)
-      (effects (font (size 1.27 1.27)) (justify right) hide)
-    )
-  )
-  (global_label "col1" (shape input) (at 35.56 55.88 180) (fields_autoplaced)
-    (effects (font (size 1.27 1.27)) (justify right))
-    (property "Intersheet References" "${INTERSHEET_REFS}" (id 0) (at 29.0345 55.9594 0)
-      (effects (font (size 1.27 1.27)) (justify right) hide)
-    )
-  )
-  (global_label "col2" (shape input) (at 129.54 109.22 180) (fields_autoplaced)
-    (effects (font (size 1.27 1.27)) (justify right))
-    (property "Intersheet References" "${INTERSHEET_REFS}" (id 0) (at 123.0145 109.1406 0)
-      (effects (font (size 1.27 1.27)) (justify right) hide)
-    )
+  (global_label "col0" (shape input) (at 35.56 48.26 180) (fields_autoplaced)
+    (effects (font (size 1.27 1.27)) (justify right))
+    (property "Intersheet References" "${INTERSHEET_REFS}" (id 0) (at 29.0345 48.1806 0)
+      (effects (font (size 1.27 1.27)) (justify right) hide)
+    )
+  )
+  (global_label "col2" (shape input) (at 35.56 60.96 180) (fields_autoplaced)
+    (effects (font (size 1.27 1.27)) (justify right))
+    (property "Intersheet References" "${INTERSHEET_REFS}" (id 0) (at 29.0345 60.8806 0)
+      (effects (font (size 1.27 1.27)) (justify right) hide)
+    )
+  )
+  (global_label "row1" (shape input) (at 35.56 55.88 180) (fields_autoplaced)
+    (effects (font (size 1.27 1.27)) (justify right))
+    (property "Intersheet References" "${INTERSHEET_REFS}" (id 0) (at 28.6717 55.8006 0)
+      (effects (font (size 1.27 1.27)) (justify right) hide)
+    )
+  )
+  (global_label "row2" (shape input) (at 129.54 109.22 180) (fields_autoplaced)
+    (effects (font (size 1.27 1.27)) (justify right))
+    (property "Intersheet References" "${INTERSHEET_REFS}" (id 0) (at 122.6517 109.1406 0)
+      (effects (font (size 1.27 1.27)) (justify right) hide)
+    )
